File: m48txx-battery-fix.sch (KiCad schematic (older format))
At the start: 4 parts, among them J1 OSC, J2 PWR, Y1 31.768kHz

Commit message: Fix a typo
Parts:
- BT1: value CR2032 -> CR2016
Changed lines of the file:
@@
 P 6000 3900
 F 0 "BT1" H 6118 3996 50  0000 L CNN
-F 1 "CR2032" H 6118 3905 50  0000 L CNN
+F 1 "CR2016" H 6118 3905 50  0000 L CNN
 F 2 "m48txx-battery-fix:BAT-HLD-002-SMT-OTL" V 6000 3960 50  0001 C CNN
 F 3 "~" V 6000 3960 50  0001 C CNN
